File: KiCAD_designs/esp_examples/esp_1st_iter_robot/esp_1st_iter_robot.kicad_sch (KiCad schematic)
At the start: 22 parts, among them J1 B2B-PH-SM4-TBLFSN, J2 B2B-PH-SM4-TBLFSN, J3 Conn_01x02_Pin, J4 Conn_01x02_Pin, J5 Conn_01x03_Pin, Q1 AO3400A, SW1 KMR223G LFG, SW2 KMR223G LFG, U1 ESP-12F, U2 AMS1117-3.3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

Commit message: esp_v3_routed with keep-out
Parts:
- removed J4: Conn_01x02_Pin, Connector_PinHeader_2.54mm:PinHeader_1x02_P2.54mm_Vertical, symbol Connector:Conn_01x02_Pin
- removed SW1, SW2: KMR223G LFG, esp_lib:KMR2_G_CNK, symbol esp_example_symbols:KMR223G_LFG
- added R6, R7: R, Resistor_SMD:R_0805_2012Metric, symbol Device:R
- added SW2, SW3: RS-282G05A3-SM RT, esp_lib:RS-282G05A3-SM RT_CNK, symbol esp_example_symbols:RS-282G05A3-SM_RT
Connections:
- net DC: now also U1.6 (GPIO12); no longer U1.16 (GPIO15)
- net GND: now also U1.16 (GPIO15), SW2.2, SW3.2; no longer R5.2
- net VCC: now also R5.2, R6.2, R7.1
- net servo: now also U1.17 (GPIO2), R6.1; no longer U1.6 (GPIO12)
- net at R1.1, U1.1 (RST): now also SW3.1
- net boot: now reaches R2.2, U1.18 (GPIO0)
- net boot: now also SW2.1
- net at U1.19 (GPIO4): no longer D1.1 (K)
- net at U1.20 (GPIO5): no longer D2.1 (K)
- net LED2: now reaches U1.4 (GPIO16)
- net LED2: now also D1.1 (K)
- net LED1: now reaches U1.5 (GPIO14)
- net LED1: now also D2.1 (K)
- net buzzer: now reaches U1.7 (GPIO13), U3.1
- net at D2.2 (A), R5.1: no longer D1.2 (A)
- new net: D1.2 (A), R7.2
Other:
- moved on the sheet: C1, C2, C3, C4, D1, D2, J1, J2, J5, Q1, R2, R3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

Commit message: esp_camRoller
Parts:
- removed J5: Conn_01x03_Pin, Connector_PinHeader_2.54mm:PinHeader_1x03_P2.54mm_Vertical, symbol Connector:Conn_01x03_Pin
- removed R6: R, Resistor_SMD:R_0805_2012Metric, symbol Device:R
- added J4: B2B-PH-SM4-TBLFSN, esp_lib:CONN_B2B-PH-SM4-TBLFSN_JST, symbol esp_example_symbols:B2B-PH-SM4-TBLFSN
- added J5: Conn_01x02_Pin, Connector_PinHeader_2.54mm:PinHeader_1x02_P2.54mm_Vertical, symbol Connector:Conn_01x02_Pin
- added Q2: AO3400A, esp_lib:SOT95P280X125-3N, symbol esp_example_symbols:AO3400A
- added R8: R, Resistor_SMD:R_0805_2012Metric, symbol Device:R
Connections:
- net GND: now also J5.1 (Pin_1), Q2.2, R8.2
- net VCC: now also J4.2
- net at C1.2, C2.2, J2.2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: now also J5.2 (Pin_2)
- net servo renamed DC2
- net DC2: now also Q2.1, R8.1
- new net: J4.1, Q2.3
Other:
- moved on the sheet: J1, Q1, R3
