File: KiCAD_designs/esp_examples/esp_1st_iter_robot/esp_1st_iter_robot.kicad_pcb (KiCad board)
At the start: 2 copper layers, 57 x 37 mm, 22 parts, among them J1 B2B-PH-SM4-TBLFSN, J2 B2B-PH-SM4-TBLFSN, J3 Conn_01x02_Pin, J4 B2B-PH-SM4-TBLFSN, J5 Conn_01x02_Pin, SW2 RS-282G05A3-SM RT, SW3 RS-282G05A3-SM RT, U1 ESP-12F, U2 AMS1117-3.3, U3 CPT-9019S-SMT-TR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

Commit message: audio
Routing:
- net /boot: track 34.6 -> 36.9 mm
Changed lines of the file:
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@@
     (fp_line (start 1 0.625) (end -1 0.625)
       (stroke (width 0.1) (type solid)) (layer "F.Fab"))
-    (pad "1" smd roundrect locked (at -0.95 0) (size 1 1.45) (layers "F.Cu" "F.Paste" "F.Mask") (roundrect_rratio 0.25)
+    (pad "1" smd roundrect (at -0.95 0) (size 1 1.45) (layers "F.Cu" "F.Paste" "F.Mask") (roundrect_rratio 0.25)
       (net 1 "GND") (pintype "passive"))
     (pad "2" smd roundrect (at 0.95 0) (size 1 1.45) (layers "F.Cu" "F.Paste" "F.Mask") (roundrect_rratio 0.25)
@@
   (segment (start 49.928634 27.635) (end 48.768 28.795634) (width 0.5) (layer "F.Cu") (net 8))
   (segment (start 48.768 31.831781) (end 46.228 34.371781) (width 0.5) (layer "F.Cu") (net 8))
+  (segment (start 83.504 28.002) (end 85.398396 28.002) (width 0.5) (layer "F.Cu") (net 9))
   (segment (start 87.63 28.002) (end 88.2885 27.3435) (width 0.5) (layer "F.Cu") (net 9))
+  (segment (start 75.692 27.051) (end 75.692 29.083) (width 0.5) (layer "F.Cu") (net 9))
   (segment (start 85.525396 28.002) (end 87.63 28.002) (width 0.5) (layer "F.Cu") (net 9))
-  (segment (start 67.818 26.289) (end 83.812396 26.289) (width 0.5) (layer "F.Cu") (net 9))
+  (segment (start 76.0657 29.4567) (end 82.0493 29.4567) (width 0.5) (layer "F.Cu") (net 9))
+  (segment (start 75.692 29.083) (end 76.0657 29.4567) (width 0.5) (layer "F.Cu") (net 9))
   (segment (start 69.214 35.635) (end 68.085 35.635) (width 0.5) (layer "F.Cu") (net 9))
-  (segment (start 83.812396 26.289) (end 85.525396 28.002) (width 0.5) (layer "F.Cu") (net 9))
+  (segment (start 67.818 26.289) (end 74.93 26.289) (width 0.5) (layer "F.Cu") (net 9))
+  (segment (start 82.0493 29.4567) (end 83.504 28.002) (width 0.5) (layer "F.Cu") (net 9))
   (segment (start 88.2885 27.3435) (end 90.424 27.3435) (width 0.5) (layer "F.Cu") (net 9))
   (segment (start 67.31 34.86) (end 67.31 26.797) (width 0.5) (layer "F.Cu") (net 9))
   (segment (start 68.085 35.635) (end 67.31 34.86) (width 0.5) (layer "F.Cu") (net 9))
   (segment (start 67.31 26.797) (end 67.818 26.289) (width 0.5) (layer "F.Cu") (net 9))
+  (segment (start 74.93 26.289) (end 75.692 27.051) (width 0.5) (layer "F.Cu") (net 9))
   (segment (start 47.752 40.8555) (end 47.436 41.1715) (width 0.5) (layer "F.Cu") (net 10))
   (segment (start 53.214 31.635) (end 50.28 31.635) (width 0.5) (layer "F.Cu") (net 10))
@@
   (segment (start 71.12 38.041) (end 71.12 44.958) (width 0.5) (layer "F.Cu") (net 12))
   (segment (start 93.7368 32.828) (end 92.3348 32.828) (width 0.762) (layer "F.Cu") (net 19))
-  (segment (start 90.667998 40.64) (end 90.967999 40.940001) (width 0.762) (layer "F.Cu") (net 19))
+  (segment (start 90.794998 40.767) (end 90.967999 40.940001) (width 0.762) (layer "F.Cu") (net 19))
   (segment (start 94.387799 40.940001) (end 90.967999 40.940001) (width 0.762) (layer "F.Cu") (net 19))
+  (segment (start 80.9058 40.1388) (end 81.534 40.767) (width 0.762) (layer "F.Cu") (net 19))
+  (segment (start 95.5784 39.7494) (end 95.5784 34.6696) (width 0.762) (layer "F.Cu") (net 19))
+  (segment (start 81.8598 32.4015) (end 81.8598 35.1955) (width 0.762) (layer "F.Cu") (net 19))
   (segment (start 80.9058 37.8195) (end 80.9058 40.1388) (width 0.762) (layer "F.Cu") (net 19))
-  (segment (start 95.5784 39.7494) (end 95.5784 34.6696) (width 0.762) (layer "F.Cu") (net 19))
-  (segment (start 81.407 40.64) (end 90.667998 40.64) (width 0.762) (layer "F.Cu") (net 19))
-  (segment (start 81.8598 32.4015) (end 81.8598 35.1955) (width 0.762) (layer "F.Cu") (net 19))
   (segment (start 95.5784 34.6696) (end 93.7368 32.828) (width 0.762) (layer "F.Cu") (net 19))
   (segment (start 80.9058 37.8195) (end 80.9058 37.404) (width 0.762) (layer "F.Cu") (net 19))
   (segment (start 81.8598 36.45) (end 81.8598 35.1955) (width 0.762) (layer "F.Cu") (net 19))
   (segment (start 80.9058 37.404) (end 81.8598 36.45) (width 0.762) (layer "F.Cu") (net 19))
-  (segment (start 80.9058 40.1388) (end 81.407 40.64) (width 0.762) (layer "F.Cu") (net 19))
+  (segment (start 81.534 40.767) (end 90.794998 40.767) (width 0.762) (layer "F.Cu") (net 19))
   (segment (start 94.387799 40.940001) (end 95.5784 39.7494) (width 0.762) (layer "F.Cu") (net 19))
   (segment (start 55.499 52.705) (end 55.499 53.709) (width 0.5) (layer "F.Cu") (net 20))
