File: KiCAD_designs/esp_examples/esp_1st_iter_robot_mistake/esp_1st_iter_robot_mistake.kicad_sch (KiCad schematic)
At the start: 22 parts, among them J1 B2B-PH-SM4-TBLFSN, J2 B2B-PH-SM4-TBLFSN, J3 Conn_01x02_Pin, J4 B2B-PH-SM4-TBLFSN, J5 Conn_01x02_Pin, SW2 RS-282G05A3-SM RT, SW3 RS-282G05A3-SM RT, U1 ESP-12F, U2 AMS1117-3.3, U3 CPT-9019S-SMT-TR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

Commit message: cam_roller_redesign
Parts:
- removed R4: R, Resistor_SMD:R_0805_2012Metric, symbol Device:R
Changed lines of the file:
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@@
   (junction (at 113.03 114.3) (diameter 0) (color 0 0 0 0)
   )
-  (junction (at 55.88 58.42) (diameter 0) (color 0 0 0 0)
-  )
   (junction (at 74.93 135.89) (diameter 0) (color 0 0 0 0)
   )
@@
     (stroke (width 0) (type default))
   )
-  (wire (pts (xy 55.88 58.42) (xy 71.12 58.42))
+  (wire (pts (xy 45.72 58.42) (xy 71.12 58.42))
     (stroke (width 0) (type default))
   )
@@
     (stroke (width 0) (type default))
   )
-  (wire (pts (xy 55.88 50.8) (xy 74.93 50.8))
-    (stroke (width 0) (type default))
-  )
   (wire (pts (xy 71.12 55.88) (xy 74.93 55.88))
     (stroke (width 0) (type default))
@@
     (stroke (width 0) (type default))
   )
-  (wire (pts (xy 45.72 58.42) (xy 55.88 58.42))
-    (stroke (width 0) (type default))
-  )
   (wire (pts (xy 242.57 41.91) (xy 248.92 41.91))
     (stroke (width 0) (type default))
@@
     (pin "1")
     (instances
-      (project "esp_1st_iter_robot"
+      (project "esp_1st_iter_robot_mistake"
         (path "/23d6f766-c6b7-4667-9a65-4887bf263ea9"
           (reference "J5") (unit 1)
@@
     (pin "1")
     (instances
-      (project "esp_1st_iter_robot"
+      (project "esp_1st_iter_robot_mistake"
         (path "/23d6f766-c6b7-4667-9a65-4887bf263ea9"
           (reference "#PWR09") (unit 1)
@@
     (pin "1")
     (instances
-      (project "esp_1st_iter_robot"
+      (project "esp_1st_iter_robot_mistake"
         (path "/23d6f766-c6b7-4667-9a65-4887bf263ea9"
           (reference "J2") (unit 1)
@@
     (pin "1")
     (instances
-      (project "esp_1st_iter_robot"
+      (project "esp_1st_iter_robot_mistake"
         (path "/23d6f766-c6b7-4667-9a65-4887bf263ea9"
           (reference "#PWR04") (unit 1)
@@
     (pin "9")
     (instances
-      (project "esp_1st_iter_robot"
+      (project "esp_1st_iter_robot_mistake"
         (path "/23d6f766-c6b7-4667-9a65-4887bf263ea9"
           (reference "U1") (unit 1)
@@
     (pin "1")
     (instances
-      (project "esp_1st_iter_robot"
+      (project "esp_1st_iter_robot_mistake"
         (path "/23d6f766-c6b7-4667-9a65-4887bf263ea9"
           (reference "#PWR07") (unit 1)
@@
     (pin "2")
     (instances
-      (project "esp_1st_iter_robot"
+      (project "esp_1st_iter_robot_mistake"
         (path "/23d6f766-c6b7-4667-9a65-4887bf263ea9"
           (reference "J4") (unit 1)
@@
     (pin "1")
     (instances
-      (project "esp_1st_iter_robot"
+      (project "esp_1st_iter_robot_mistake"
         (path "/23d6f766-c6b7-4667-9a65-4887bf263ea9"
           (reference "#PWR06") (unit 1)
@@
     (pin "1")
     (instances
-      (project "esp_1st_iter_robot"
+      (project "esp_1st_iter_robot_mistake"
         (path "/23d6f766-c6b7-4667-9a65-4887bf263ea9"
           (reference "U2") (unit 1)
@@
     (pin "2")
     (instances
-      (project "esp_1st_iter_robot"
+      (project "esp_1st_iter_robot_mistake"
         (path "/23d6f766-c6b7-4667-9a65-4887bf263ea9"
           (reference "D1") (unit 1)
@@
     (pin "1")
     (instances
-      (project "esp_1st_iter_robot"
+      (project "esp_1st_iter_robot_mistake"
         (path "/23d6f766-c6b7-4667-9a65-4887bf263ea9"
           (reference "R5") (unit 1)
@@
     (pin "2")
     (instances
-      (project "esp_1st_iter_robot"
+      (project "esp_1st_iter_robot_mistake"
         (path "/23d6f766-c6b7-4667-9a65-4887bf263ea9"
           (reference "U3") (unit 1)
@@
     (pin "2")
     (instances
-      (project "esp_1st_iter_robot"
+      (project "esp_1st_iter_robot_mistake"
         (path "/23d6f766-c6b7-4667-9a65-4887bf263ea9"
           (reference "R1") (unit 1)
@@
     (pin "2")
     (instances
-      (project "esp_1st_iter_robot"
+      (project "esp_1st_iter_robot_mistake"
         (path "/23d6f766-c6b7-4667-9a65-4887bf263ea9"
           (reference "SW2") (unit 1)
@@
     (pin "2")
     (instances
-      (project "esp_1st_iter_robot"
+      (project "esp_1st_iter_robot_mistake"
         (path "/23d6f766-c6b7-4667-9a65-4887bf263ea9"
           (reference "C2") (unit 1)
@@
     (pin "1")
     (instances
-      (project "esp_1st_iter_robot"
+      (project "esp_1st_iter_robot_mistake"
         (path "/23d6f766-c6b7-4667-9a65-4887bf263ea9"
           (reference "#PWR05") (unit 1)
@@
     (pin "1")
     (instances
-      (project "esp_1st_iter_robot"
+      (project "esp_1st_iter_robot_mistake"
         (path "/23d6f766-c6b7-4667-9a65-4887bf263ea9"
           (reference "C1") (unit 1)
@@
     (pin "1")
     (instances
-      (project "esp_1st_iter_robot"
+      (project "esp_1st_iter_robot_mistake"
         (path "/23d6f766-c6b7-4667-9a65-4887bf263ea9"
           (reference "#PWR014") (unit 1)
@@
     (pin "1")
     (instances
-      (project "esp_1st_iter_robot"
+      (project "esp_1st_iter_robot_mistake"
         (path "/23d6f766-c6b7-4667-9a65-4887bf263ea9"
           (reference "#PWR015") (unit 1)
@@
     (pin "1")
     (instances
-      (project "esp_1st_iter_robot"
+      (project "esp_1st_iter_robot_mistake"
         (path "/23d6f766-c6b7-4667-9a65-4887bf263ea9"
           (reference "#PWR01") (unit 1)
@@
     (pin "1")
     (instances
-      (project "esp_1st_iter_robot"
+      (project "esp_1st_iter_robot_mistake"
         (path "/23d6f766-c6b7-4667-9a65-4887bf263ea9"
           (reference "#PWR010") (unit 1)
@@
     (pin "1")
     (instances
-      (project "esp_1st_iter_robot"
+      (project "esp_1st_iter_robot_mistake"
         (path "/23d6f766-c6b7-4667-9a65-4887bf263ea9"
           (reference "R2") (unit 1)
@@
     (pin "1")
     (instances
-      (project "esp_1st_iter_robot"
+      (project "esp_1st_iter_robot_mistake"
         (path "/23d6f766-c6b7-4667-9a65-4887bf263ea9"
           (reference "#PWR02") (unit 1)
@@
     (pin "1")
     (instances
-      (project "esp_1st_iter_robot"
+      (project "esp_1st_iter_robot_mistake"
         (path "/23d6f766-c6b7-4667-9a65-4887bf263ea9"
           (reference "#PWR03") (unit 1)
@@
     (pin "2")
     (instances
-      (project "esp_1st_iter_robot"
+      (project "esp_1st_iter_robot_mistake"
         (path "/23d6f766-c6b7-4667-9a65-4887bf263ea9"
           (reference "D2") (unit 1)
@@
     (pin "1")
     (instances
-      (project "esp_1st_iter_robot"
+      (project "esp_1st_iter_robot_mistake"
         (path "/23d6f766-c6b7-4667-9a65-4887bf263ea9"
           (reference "#PWR08") (unit 1)
@@
     (pin "2")
     (instances
-      (project "esp_1st_iter_robot"
+      (project "esp_1st_iter_robot_mistake"
         (path "/23d6f766-c6b7-4667-9a65-4887bf263ea9"
           (reference "J1") (unit 1)
@@
     )
   )
-  (symbol (lib_id "Device:R") (at 55.88 54.61 0) (unit 1)
-    (in_bom yes) (on_board yes) (dnp no) (fields_autoplaced)
-    (property "Reference" "R4" (at 58.42 53.34 0)
-      (effects (font (size 1.27 1.27)) (justify left))
-    )
-    (property "Value" "R" (at 58.42 55.88 0)
-      (effects (font (size 1.27 1.27)) (justify left))
-    )
-    (property "Footprint" "Resistor_SMD:R_0805_2012Metric" (at 54.102 54.61 90)
-      (effects (font (size 1.27 1.27)) hide)
-    )
-    (property "Datasheet" "~" (at 55.88 54.61 0)
-      (effects (font (size 1.27 1.27)) hide)
-    )
-    (pin "1")
-    (pin "2")
-    (instances
-      (project "esp_1st_iter_robot"
-        (path "/23d6f766-c6b7-4667-9a65-4887bf263ea9"
-          (reference "R4") (unit 1)
-        )
-      )
-    )
-  )
   (symbol (lib_id "Device:C") (at 264.16 44.45 0) (unit 1)
     (in_bom yes) (on_board yes) (dnp no) (fields_autoplaced)
@@
     (pin "1")
     (instances
-      (project "esp_1st_iter_robot"
+      (project "esp_1st_iter_robot_mistake"
         (path "/23d6f766-c6b7-4667-9a65-4887bf263ea9"
           (reference "C4") (unit 1)
@@
     (pin "1")
     (instances
-      (project "esp_1st_iter_robot"
+      (project "esp_1st_iter_robot_mistake"
         (path "/23d6f766-c6b7-4667-9a65-4887bf263ea9"
           (reference "#PWR013") (unit 1)
@@
     (pin "2")
     (instances
-      (project "esp_1st_iter_robot"
+      (project "esp_1st_iter_robot_mistake"
         (path "/23d6f766-c6b7-4667-9a65-4887bf263ea9"
           (reference "C3") (unit 1)
@@
     (pin "1")
     (instances
-      (project "esp_1st_iter_robot"
+      (project "esp_1st_iter_robot_mistake"
         (path "/23d6f766-c6b7-4667-9a65-4887bf263ea9"
           (reference "J3") (unit 1)
@@
     (pin "9-UB")
     (instances
-      (project "esp_1st_iter_robot"
+      (project "esp_1st_iter_robot_mistake"
         (path "/23d6f766-c6b7-4667-9a65-4887bf263ea9"
           (reference "U4") (unit 1)
@@
     (pin "1")
     (instances
-      (project "esp_1st_iter_robot"
+      (project "esp_1st_iter_robot_mistake"
         (path "/23d6f766-c6b7-4667-9a65-4887bf263ea9"
           (reference "SW3") (unit 1)
@@
     (pin "2")
     (instances
-      (project "esp_1st_iter_robot"
+      (project "esp_1st_iter_robot_mistake"
         (path "/23d6f766-c6b7-4667-9a65-4887bf263ea9"
           (reference "R7") (unit 1)
