File: KiCAD_designs/esp_examples/esp_thermalCam/esp_thermalCam.kicad_sch (KiCad schematic)
At the start: 22 parts, among them J1 B2B-PH-SM4-TBLFSN, J2 B2B-PH-SM4-TBLFSN, J3 Conn_01x02_Pin, J4 B2B-PH-SM4-TBLFSN, J5 Conn_01x02_Pin, SW2 RS-282G05A3-SM RT, SW3 RS-282G05A3-SM RT, U1 ESP-12F, U2 AMS1117-3.3, U3 CPT-9019S-SMT-TR, U4 MX1508

Commit message: espboy_full
Parts:
- removed D1, D2: LED, LED_SMD:LED_1206_3216Metric, symbol Device:LED
- removed J1, J4: B2B-PH-SM4-TBLFSN, esp_lib:CONN_B2B-PH-SM4-TBLFSN_JST, symbol esp_example_symbols:B2B-PH-SM4-TBLFSN
- removed R5, R7: R, Resistor_SMD:R_0805_2012Metric, symbol Device:R
- removed U3: CPT-9019S-SMT-TR, esp_lib:SM_CPT_9X9_CUD, symbol esp_example_symbols:CPT-9019S-SMT-TR
- removed U4: MX1508, esp_lib:MX1508, symbol esp_example_symbols:MX1508
- added J1, J4: B4B-ZR-SM4-TFT_LF__SN_, esp_lib:JST_B4B-ZR-SM4-TFT_LF__SN_, symbol esp_example_symbols:B4B-ZR-SM4-TFT_LF__SN_
- added J6: B7B-ZR-SM4-TFT_LF__SN_, esp_lib:B7B-ZR-SM4-TBLFSN_JST, symbol esp_example_symbols:B7B-ZR-SM4-TFT_LF__SN_
- added S1: up, esp_lib:switch, symbol esp_example_symbols:switch
- added S2: down, esp_lib:switch, symbol esp_example_symbols:switch
- added S3: left, esp_lib:switch, symbol esp_example_symbols:switch
- added S4: right, esp_lib:switch, symbol esp_example_symbols:switch
- added S5: A, esp_lib:switch, symbol esp_example_symbols:switch
- added S6: B, esp_lib:switch, symbol esp_example_symbols:switch
- added S7: RL, esp_lib:switch, symbol esp_example_symbols:switch
- added S8: RR, esp_lib:switch, symbol esp_example_symbols:switch
- added U3: MCP23017-E_SO, esp_lib:MCP23017, symbol esp_example_symbols:MCP23017-E_SO
- J2: footprint esp_lib:CONN_B2B-PH-SM4-TBLFSN_JST -> esp_lib:B2B-PH-SM4-TBLFSN_JST
Connections:
- net GND: now also J1.2, J4.2, J6.1, S1.1, S1.3, S2.1, S2.3, S3.1, S3.3, S4.1, S4.3, S5.1, S5.3, S6.1, S6.3, S7.1, S7.3, S8.1, S8.3, U3.10 (VSS)
- net VCC: now also J1.1, J4.1, J6.6, U3.18 (~{RESET}), U3.9 (VDD)
- net RST: now reaches R1.1, SW3.1, U1.1 (RST)
- net RST: now also J6.7
- net LED1 renamed SDA_mcp
- net SDA_mcp: now also J1.4, J4.4, U3.13 (SDA)
- net LED2 renamed SCK_mcp
- net SCK_mcp: now also J1.3, J4.3, U3.12 (SCK)
- net buzzer: no longer names the net of U1.17 (GPIO2)
- net in1 renamed SDA_screen
- net SDA_screen: now also J6.4
- net in2 renamed AO
- net AO: now also J6.5
- net in3 renamed SCK_screen
- net SCK_screen: now also J6.2
- net in4 renamed CS
- net CS: now also J6.3
- new net: J4.S1 (SHIELD), J4.S2 (SHIELD)
- new net: J1.S1 (SHIELD), J1.S2 (SHIELD)
- new net A: S5.4, U3.28 (GPA7)
- new net B: S6.4, U3.27 (GPA6)
- new net RL: S7.2, U3.22 (GPA1)
- new net RR: S8.4, U3.21 (GPA0)
- new net down: S2.2, U3.26 (GPA5)
- new net left: S3.4, U3.23 (GPA2)
- new net right: S4.4, U3.25 (GPA4)
- new net up: S1.4, U3.24 (GPA3)
