File: KiCAD_designs/esp_examples/esp_audio/esp_audio.kicad_pcb (KiCad board)
At the start: 2 copper layers, 57 x 33 mm, 24 parts, among them J1 B2B-PH-SM4-TBLFSN, J2 B2B-PH-SM4-TBLFSN, J3 Conn_01x02_Pin, J5 Conn_01x02_Pin, P1 S3B-ZR-SM4A-TF, SW1 RS-282G05A3-SM RT, SW2 RS-282G05A3-SM RT, SW3 RS-282G05A3-SM RT, U1 ESP-12F, U2 AMS1117-3.3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

Commit message: design-cleanup
Routing:
- net GND: track 5.59 -> 0.00 mm
Changed lines of the file:
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@@
     (style (thickness 0.15) (arrow_length 1.27) (text_position_mode 0) (extension_height 0.58642) (extension_offset 0.5) keep_text_aligned)
   )
-  (segment (start 79.9598 32.4015) (end 79.9598 35.1955) (width 0.5) (layer "F.Cu") (net 1))
-  (segment (start 86.1778 32.32) (end 86.1778 35.114) (width 0.5) (layer "F.Cu") (net 1))
   (segment (start 44.717 40.1575) (end 44.717 42.418) (width 0.762) (layer "F.Cu") (net 2))
   (segment (start 46.228 37.3615) (end 46.228 39.0925) (width 0.762) (layer "F.Cu") (net 2))
