File: KiCAD_designs/esp_examples/esp_espboy/esp_espboy.kicad_pcb (KiCad board)
At the start: 2 copper layers, 57 x 37 mm, 22 parts, among them J1 B2B-PH-SM4-TBLFSN, J2 B2B-PH-SM4-TBLFSN, J3 Conn_01x02_Pin, J4 B2B-PH-SM4-TBLFSN, J5 Conn_01x02_Pin, SW2 RS-282G05A3-SM RT, SW3 RS-282G05A3-SM RT, U1 ESP-12F, U2 AMS1117-3.3, U3 CPT-9019S-SMT-TR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

Commit message: espboy_copy
Parts:
- removed D1, D2: LED, LED_SMD:LED_1206_3216Metric
- removed R5, R7: R, Resistor_SMD:R_0805_2012Metric
- removed U4: MX1508, esp_lib:MX1508
- added J6: B7B-ZR-SM4-TFT_LF__SN_, esp_lib:B7B-ZR-SM4-TBLFSN_JST, F.Cu at (59.2, 51.8)
- added S1: up, esp_lib:switch, F.Cu at (47.0, 81.9)
- added S2: down, esp_lib:switch, F.Cu at (47.0, 88.0)
- added S3: left, esp_lib:switch, F.Cu at (42.9, 85.0)
- added S4: right, esp_lib:switch, F.Cu at (51.1, 85.0)
- added S5: A, esp_lib:switch, F.Cu at (89.7, 86.0)
- added S6: B, esp_lib:switch, F.Cu at (94.0, 82.2)
- added S7: RL, esp_lib:switch, F.Cu at (47.4, 68.3)
- added S8: RR, esp_lib:switch, F.Cu at (89.2, 68.2)
- J1, J4: value B2B-PH-SM4-TBLFSN -> B4B-ZR-SM4-TFT_LF__SN_; footprint esp_lib:CONN_B2B-PH-SM4-TBLFSN_JST -> esp_lib:JST_B4B-ZR-SM4-TFT_LF__SN_
- J2: footprint esp_lib:CONN_B2B-PH-SM4-TBLFSN_JST -> esp_lib:B2B-PH-SM4-TBLFSN_JST
- U3: value CPT-9019S-SMT-TR -> MCP23017-E_SO; footprint esp_lib:SM_CPT_9X9_CUD -> esp_lib:MCP23017
- moved J4 40.4 mm to (68.9, 90.5), turned to 180 degrees
- moved U3 32.3 mm to (68.9, 76.9), turned to 180 degrees
- moved J1 19.1 mm to (82.1, 53.6), turned to 180 degrees
Connections:
- net Net-(U1-RST) renamed /RST
- J1 pad 1: Net-(U4A-OUTA1) -> VCC
- J1 pad 2: Net-(U4A-OUTB1) -> GND
- J1 pad 3: (no net) -> /SCK_mcp
- J1 pad 4: (no net) -> /SDA_mcp
- J4 pad 1: Net-(U4A-OUTA2) -> VCC
- J4 pad 2: Net-(U4A-OUTB2) -> GND
- J4 pad 3: (no net) -> /SCK_mcp
- J4 pad 4: (no net) -> /SDA_mcp
- U1 pad 17: /buzzer -> unconnected-(U1-GPIO2-Pad17)
- U1 pad 19: /LED1 -> /SDA_mcp
- U1 pad 20: /LED2 -> /SCK_mcp
- U1 pad 4: /in2 -> /AO
- U1 pad 5: /in1 -> /SDA_screen
- U1 pad 6: /in4 -> /CS
- U1 pad 7: /in3 -> /SCK_screen
- U3 pad 1: /buzzer -> unconnected-(U3-GPB0-Pad1)
- U3 pad 2: GND -> unconnected-(U3-GPB1-Pad2)
Routing:
- net /B: track 0.00 -> 53.9 mm
- net /SCK_mcp: track 0.00 -> 49.6 mm
- net /SDA_mcp: track 0.00 -> 47.8 mm
- net /RR: track 0.00 -> 43.6 mm
- net /A: track 0.00 -> 40.3 mm
- net Net-(U4A-OUTB2): track 35.5 -> 0.00 mm
- net /RL: track 0.00 -> 29.1 mm
- net Net-(U4A-OUTA2): track 29.0 -> 0.00 mm
- net /left: track 0.00 -> 26.6 mm
- net /AO: track 0.00 -> 26.5 mm
- net /SDA_screen: track 0.00 -> 25.3 mm
- net /buzzer: track 25.2 -> 0.00 mm
- net /CS: track 0.00 -> 23.3 mm
- net /SCK_screen: track 0.00 -> 21.8 mm
- net /down: track 0.00 -> 20.4 mm
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Other:
- board size 57 x 37 mm -> 57 x 72 mm

Commit message: larger button boy
Parts:
- removed S7: RL, esp_lib:switch
- removed S8: RR, esp_lib:switch
- added SW1: D2FS-FL-N-A, esp_lib:D2FS-FL-N-A_OMR, F.Cu at (54.4, 72.4)
- added SW4: D2FS-FL-N-A, esp_lib:D2FS-FL-N-A_OMR, F.Cu at (109.1, 72.4)
- S1, S2, S3, S4, S5, S6: footprint esp_lib:switch -> esp_lib:switch_6
- moved J4 34.5 mm to (103.3, 92.7)
- moved S6 14.5 mm to (107.6, 77.2), turned to 0 degrees
- moved S5 13.1 mm to (102.6, 84.1), turned to 180 degrees
- moved U3 10.2 mm to (78.0, 72.2), turned to -90 degrees
- moved S4 8.28 mm to (59.3, 84.3), turned to 180 degrees
- moved S1 7.48 mm to (53.0, 77.4), turned to 0 degrees
- moved S2 6.98 mm to (53.2, 91.2), turned to 180 degrees
- moved S3 3.81 mm to (46.7, 84.3), turned to 180 degrees
Routing:
- net VCC: track 213.8 -> 250.7 mm
- net /SCK_mcp: track 49.6 -> 75.1 mm
- net /A: track 40.3 -> 15.3 mm
- net /RR: track 43.6 -> 67.8 mm
- net /SDA_mcp: track 47.8 -> 71.2 mm
- net /right: track 14.0 -> 34.1 mm
- net /left: track 26.6 -> 46.0 mm
- net /RL: track 29.1 -> 44.0 mm
- net /down: track 20.4 -> 34.1 mm
- net /up: track 19.6 -> 28.8 mm
- net /B: track 53.9 -> 55.7 mm
Other:
- board size 57 x 72 mm -> 74.5 x 72 mm
