File: KiCAD_designs/esp_examples/esp_espboy/esp_espboy.kicad_sch (KiCad schematic)
At the start: 23 parts, among them J2 B2B-PH-SM4-TBLFSN, J3 Conn_01x02_Pin, J5 Conn_01x02_Pin, SW2 RS-282G05A3-SM RT, SW3 RS-282G05A3-SM RT, U1 ESP-12F, U2 AMS1117-3.3, U3 MCP23017-E_SO

Commit message: espboy_full
Parts:
- added J1, J4: B4B-ZR-SM4-TFT_LF__SN_, symbol esp_example_symbols:B4B-ZR-SM4-TFT_LF__SN_
- added J6, J7: B7B-ZR-SM4-TFT_LF__SN_, symbol esp_example_symbols:B7B-ZR-SM4-TFT_LF__SN_
Connections:
- net GND: now also U3.10 (VSS), J1.1, J4.4, J6.6, J7.6
- net VCC: now also U3.18 (~{RESET}), U3.9 (VDD), J1.4, J4.1, J6.7, J7.7
- net SCL: now reaches U3.12 (SCK)
- net SCL: now also U1.20 (GPIO5), J1.2, J4.3
- net SDA: now reaches U3.13 (SDA)
- net SDA: now also U1.19 (GPIO4), J1.3, J4.2
- net RST: now reaches R1.1, SW3.1, U1.1 (RST)
- net RST: now also J6.4, J7.4
- net AO: now reaches U1.17 (GPIO2)
- net AO: now also J6.3, J7.3
- net SDA_screen: now reaches U1.5 (GPIO14)
- net SDA_screen: now also J6.2, J7.2
- net CS: now reaches U1.6 (GPIO12)
- net CS: now also J6.5, J7.5
- net SCK: now reaches U1.7 (GPIO13)
- net SCK: now also J6.1, J7.1
- new net: J1.S1 (SHIELD), J1.S2 (SHIELD)
- new net: J4.S1 (SHIELD), J4.S2 (SHIELD)

Commit message: espboy_copy
Parts:
- removed J7: B7B-ZR-SM4-TFT_LF__SN_, symbol esp_example_symbols:B7B-ZR-SM4-TFT_LF__SN_
- J1, J4: footprint (none) -> esp_lib:JST_B4B-ZR-SM4-TFT_LF__SN_
- J2: footprint esp_lib:CONN_B2B-PH-SM4-TBLFSN_JST -> esp_lib:B2B-PH-SM4-TBLFSN_JST
- J6: footprint (none) -> esp_lib:B7B-ZR-SM4-TBLFSN_JST
- S1, S5, S6: footprint (none) -> esp_lib:switch
- S2: value left -> down; footprint (none) -> esp_lib:switch
- S3: value right -> left; footprint (none) -> esp_lib:switch
- S4: value down -> right; footprint (none) -> esp_lib:switch
- S7: value L -> RL; footprint (none) -> esp_lib:switch
- S8: value R -> RR; footprint (none) -> esp_lib:switch
- U3: footprint (none) -> esp_lib:MCP23017
Connections:
- net AO: now also J6.5, U1.4 (GPIO16); no longer J6.3, U1.17 (GPIO2)
- net CS: now also J6.3; no longer J6.5
- net GND: now also J1.2, J4.2, J6.1, S1.1, S1.3, S2.1, S2.3, S3.1, S3.3, S4.1, S4.3, S5.1, S5.3, S6.1, S6.3, S7.1, S7.3, S8.1, S8.3; no longer J1.1, J4.4, J6.6
- net RST: now also J6.7; no longer J6.4
- net SDA_screen: now also J6.4; no longer J6.2
- net VCC: now also J1.1, J6.6; no longer J1.4, J6.7
- net boot: now also U1.18 (GPIO0)
- net RR: now reaches U3.21 (GPA0)
- net RR: now also S8.4
- net RL: now reaches U3.22 (GPA1)
- net RL: now also S7.2
- net left: now reaches U3.23 (GPA2)
- net left: now also S3.4
- net up: now reaches U3.24 (GPA3)
- net up: now also S1.4
- net right: now reaches U3.25 (GPA4)
- net right: now also S4.4
- net down: now reaches U3.26 (GPA5)
- net down: now also S2.2
- net B: now reaches U3.27 (GPA6)
- net B: now also S6.4
- net A: now reaches U3.28 (GPA7)
- net A: now also S5.4
- net SCK renamed SCK_screen
- net SCK_screen: now also J6.2; no longer J6.1
- net SCL renamed SCK_mcp
- net SCK_mcp: now also J1.3; no longer J1.2
- net SDA renamed SDA_mcp
- net SDA_mcp: now also J1.4, J4.4; no longer J1.3, J4.2
Other:
- moved on the sheet: C1, C2, C3, C4, J2, J3, J5, R1, R2, R4, SW2, SW3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

Commit message: larger button boy
Parts:
- removed S7: RL, esp_lib:switch, symbol esp_example_symbols:switch
- removed S8: RR, esp_lib:switch, symbol esp_example_symbols:switch
- added SW1, SW4: D2FS-FL-N-A, D2FS-FL-N-A_OMR, symbol esp_example_symbols:D2FS-FL-N-A
- S1, S2, S3, S4, S5, S6: footprint esp_lib:switch -> esp_lib:switch_6
Connections:
- net GND: now also SW1.1, SW1.3, SW4.1, SW4.3
- net RL: now also SW1.2
- net RR: now also SW4.2
