File: KiCAD_designs/esp_examples/App_espboy/App_espboy.kicad_pcb (KiCad board)
At the start: 2 copper layers, 74.5 x 72 mm, 32 parts, among them J1 B4B-ZR-SM4-TFT_LF__SN_, J2 B2B-PH-SM4-TBLFSN, J3 Conn_01x02_Pin, J4 B4B-ZR-SM4-TFT_LF__SN_, J5 Conn_01x02_Pin, J6 B7B-ZR-SM4-TFT_LF__SN_, SW1 D2FS-FL-N-A, SW2 RS-282G05A3-SM RT, SW3 RS-282G05A3-SM RT, SW4 D2FS-FL-N-A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

Commit message: 23017
Parts:
- removed C5: C, Capacitor_SMD:C_0805_2012Metric
- removed R3, R5, R6, R7, R8: R, Resistor_SMD:R_0805_2012Metric
- moved U3 5.23 mm to (78.0, 72.2)
- moved SW1 3.84 mm to (58.2, 72.4)
Connections:
- SW1 pad 1: GND -> unconnected-(SW1-Pad1)
- SW4 pad 1: GND -> unconnected-(SW4-Pad1)
- U3 pad 15: GND -> unconnected-(U3-A0-Pad15)
- U3 pad 16: GND -> unconnected-(U3-A1-Pad16)
- U3 pad 17: GND -> unconnected-(U3-A2-Pad17)
- U3 pad 18: Net-(U3-~{RESET}) -> VCC
- U3 pad 19: Net-(U3-INTB) -> unconnected-(U3-INTB-Pad19)
- U3 pad 20: Net-(U3-INTA) -> unconnected-(U3-INTA-Pad20)
Routing:
- net Net-(U3-INTA): track 18.1 -> 0.00 mm
- net Net-(U3-INTB): track 17.6 -> 0.00 mm
- net Net-(U3-~{RESET}): track 16.5 -> 0.00 mm
- net VCC: track 237.1 -> 250.7 mm
- net /RL: track 53.4 -> 40.5 mm
- net /RR: track 78.1 -> 67.8 mm
- net /up: track 37.2 -> 28.8 mm
- net /left: track 53.9 -> 46.0 mm
- net /right: track 41.6 -> 34.1 mm
- net /down: track 40.7 -> 34.1 mm
- net /B: track 50.1 -> 55.7 mm
- net /A: track 9.86 -> 15.3 mm
- net /SDA_mcp: track 72.3 -> 71.2 mm
- net /SCK_mcp: track 76.0 -> 75.1 mm
Other:
- outline, holes or cut-outs redrawn
