File: KiCAD_designs/esp_examples/App_boy/App_boy.kicad_pcb (KiCad board)
At the start: 2 copper layers, 74.5 x 72 mm, 26 parts, among them J1 B4B-ZR-SM4-TFT_LF__SN_, J2 B2B-PH-SM4-TBLFSN, J3 Conn_01x02_Pin, J4 B4B-ZR-SM4-TFT_LF__SN_, J5 Conn_01x02_Pin, J6 B7B-ZR-SM4-TFT_LF__SN_, SW1 D2FS-FL-N-A, SW2 RS-282G05A3-SM RT, SW3 RS-282G05A3-SM RT, SW4 D2FS-FL-N-A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

Commit message: 23017 Updated
Parts:
- added C5: C, Capacitor_SMD:C_0805_2012Metric, F.Cu at (83.8, 66.3)
- added R3: R, Resistor_SMD:R_0805_2012Metric, F.Cu at (69.4, 67.7)
- added R5: R, Resistor_SMD:R_0805_2012Metric, F.Cu at (69.4, 69.8)
- added R6: R, Resistor_SMD:R_0805_2012Metric, F.Cu at (69.4, 76.0)
- added R7: R, Resistor_SMD:R_0805_2012Metric, F.Cu at (69.4, 73.9)
- added R8: R, Resistor_SMD:R_0805_2012Metric, F.Cu at (69.4, 71.8)
- moved U3 5.23 mm to (83.0, 73.6)
- moved SW1 3.84 mm to (54.4, 72.4)
Connections:
- SW1 pad 1: unconnected-(SW1-Pad1) -> GND
- SW4 pad 1: unconnected-(SW4-Pad1) -> GND
- U3 pad 15: unconnected-(U3-A0-Pad15) -> GND
- U3 pad 16: unconnected-(U3-A1-Pad16) -> GND
- U3 pad 17: unconnected-(U3-A2-Pad17) -> GND
- U3 pad 18: VCC -> Net-(U3-~{RESET})
- U3 pad 19: unconnected-(U3-INTB-Pad19) -> Net-(U3-INTB)
- U3 pad 20: unconnected-(U3-INTA-Pad20) -> Net-(U3-INTA)
Routing:
- net Net-(U3-INTA): track 0.00 -> 18.1 mm
- net Net-(U3-INTB): track 0.00 -> 17.6 mm
- net Net-(U3-~{RESET}): track 0.00 -> 16.5 mm
- net /RL: track 40.5 -> 53.4 mm
- net /RR: track 67.8 -> 78.1 mm
- net /up: track 28.8 -> 37.2 mm
- net /left: track 46.0 -> 53.9 mm
- net /right: track 34.1 -> 41.6 mm
- net /down: track 34.1 -> 40.7 mm
- net /B: track 55.7 -> 50.1 mm
- net /A: track 15.3 -> 9.86 mm
- net VCC: track 250.7 -> 245.5 mm
- net /SDA_mcp: track 71.2 -> 72.3 mm
- net /SCK_mcp: track 75.1 -> 76.0 mm
Other:
- outline, holes or cut-outs redrawn
