File: KiCAD_designs/esp_examples/App_boy/App_boy.kicad_sch (KiCad schematic)
At the start: 26 parts, among them J1 B4B-ZR-SM4-TFT_LF__SN_, J2 B2B-PH-SM4-TBLFSN, J3 Conn_01x02_Pin, J4 B4B-ZR-SM4-TFT_LF__SN_, J5 Conn_01x02_Pin, J6 B7B-ZR-SM4-TFT_LF__SN_, SW1 D2FS-FL-N-A, SW2 RS-282G05A3-SM RT, SW3 RS-282G05A3-SM RT, SW4 D2FS-FL-N-A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

Commit message: 23017 Updated
Parts:
- added C5: C, Capacitor_SMD:C_0805_2012Metric, symbol Device:C
- added R3, R5, R6, R7, R8: R, Resistor_SMD:R_0805_2012Metric, symbol Device:R
Connections:
- net GND: now also U3.15 (A0), U3.16 (A1), U3.17 (A2), C5.1
- net SCK_mcp: now also R3.2
- net SDA_mcp: now also R5.2
- net VCC: now also C5.2, R3.1, R5.1, R6.2, R7.2, R8.2; no longer U3.18 (~{RESET})
- net at U3.19 (INTB): now also R7.1
- net at U3.20 (INTA): now also R6.1
- new net: R8.1, U3.18 (~{RESET})
Changed lines of the file:
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@@
   (junction (at 264.16 48.26) (diameter 0) (color 0 0 0 0)
   )
+  (junction (at 22.86 172.72) (diameter 0) (color 0 0 0 0)
+  )
+  (junction (at 71.12 170.18) (diameter 0) (color 0 0 0 0)
+  )
+  (junction (at 71.12 172.72) (diameter 0) (color 0 0 0 0)
+  )
   (junction (at 220.98 22.86) (diameter 0) (color 0 0 0 0)
   )
@@
   (junction (at 55.88 58.42) (diameter 0) (color 0 0 0 0)
   )
+  (junction (at 58.42 182.88) (diameter 0) (color 0 0 0 0)
+  )
+  (junction (at 22.86 170.18) (diameter 0) (color 0 0 0 0)
+  )
   (junction (at 45.72 48.26) (diameter 0) (color 0 0 0 0)
   )
@@
     (stroke (width 0) (type default))
   )
+  (wire (pts (xy 71.12 182.88) (xy 66.04 182.88))
+    (stroke (width 0) (type default))
+  )
   (wire (pts (xy 113.03 50.8) (xy 110.49 50.8))
     (stroke (width 0) (type default))
@@
     (stroke (width 0) (type default))
   )
+  (wire (pts (xy 71.12 170.18) (xy 71.12 172.72))
+    (stroke (width 0) (type default))
+  )
   (wire (pts (xy 156.21 45.72) (xy 160.02 45.72))
     (stroke (width 0) (type default))
@@
     (stroke (width 0) (type default))
   )
+  (wire (pts (xy 22.86 139.7) (xy 19.05 139.7))
+    (stroke (width 0) (type default))
+  )
+  (wire (pts (xy 58.42 170.18) (xy 63.5 170.18))
+    (stroke (width 0) (type default))
+  )
   (wire (pts (xy 248.92 48.26) (xy 255.27 48.26))
     (stroke (width 0) (type default))
@@
     (stroke (width 0) (type default))
   )
+  (wire (pts (xy 22.86 182.88) (xy 58.42 182.88))
+    (stroke (width 0) (type default))
+  )
+  (wire (pts (xy 71.12 167.64) (xy 71.12 170.18))
+    (stroke (width 0) (type default))
+  )
   (wire (pts (xy 55.88 58.42) (xy 71.12 58.42))
     (stroke (width 0) (type default))
@@
     (stroke (width 0) (type default))
   )
+  (wire (pts (xy 58.42 182.88) (xy 58.42 177.8))
+    (stroke (width 0) (type default))
+  )
+  (wire (pts (xy 71.12 172.72) (xy 71.12 182.88))
+    (stroke (width 0) (type default))
+  )
   (wire (pts (xy 229.87 22.86) (xy 229.87 25.4))
     (stroke (width 0) (type default))
   )
+  (wire (pts (xy 58.42 167.64) (xy 63.5 167.64))
+    (stroke (width 0) (type default))
+  )
   (wire (pts (xy 76.2 30.48) (xy 76.2 34.29))
     (stroke (width 0) (type default))
@@
     (stroke (width 0) (type default))
   )
+  (wire (pts (xy 58.42 172.72) (xy 63.5 172.72))
+    (stroke (width 0) (type default))
+  )
   (wire (pts (xy 212.09 30.48) (xy 212.09 41.91))
     (stroke (width 0) (type default))
   )
+  (wire (pts (xy 22.86 167.64) (xy 22.86 170.18))
+    (stroke (width 0) (type default))
+  )
+  (wire (pts (xy 22.86 170.18) (xy 22.86 172.72))
+    (stroke (width 0) (type default))
+  )
   (wire (pts (xy 248.92 48.26) (xy 248.92 46.99))
     (stroke (width 0) (type default))
@@
     (stroke (width 0) (type default))
   )
+  (wire (pts (xy 19.05 128.27) (xy 19.05 139.7))
+    (stroke (width 0) (type default))
+  )
+  (wire (pts (xy 22.86 172.72) (xy 22.86 182.88))
+    (stroke (width 0) (type default))
+  )
   (wire (pts (xy 187.96 45.72) (xy 193.04 45.72))
     (stroke (width 0) (type default))
@@
   )
   (wire (pts (xy 45.72 58.42) (xy 55.88 58.42))
+    (stroke (width 0) (type default))
+  )
+  (wire (pts (xy 22.86 128.27) (xy 22.86 137.16))
     (stroke (width 0) (type default))
   )
@@
     (effects (font (size 1.27 1.27)) (justify right bottom))
   )
+  (label "VCC" (at 22.86 120.65 0) (fields_autoplaced)
+    (effects (font (size 1.27 1.27)) (justify left bottom))
+  )
   (label "boot" (at 151.13 45.72 0) (fields_autoplaced)
     (effects (font (size 1.27 1.27)) (justify left bottom))
@@
     (effects (font (size 1.27 1.27)) (justify right bottom))
   )
-  (label "VCC" (at 58.42 172.72 0) (fields_autoplaced)
+  (label "VCC" (at 71.12 167.64 0) (fields_autoplaced)
     (effects (font (size 1.27 1.27)) (justify left bottom))
   )
@@
   (label "AO" (at 74.93 83.82 180) (fields_autoplaced)
     (effects (font (size 1.27 1.27)) (justify right bottom))
+  )
+  (label "VCC" (at 19.05 120.65 0) (fields_autoplaced)
+    (effects (font (size 1.27 1.27)) (justify left bottom))
   )
   (label "RST" (at 231.14 93.98 270) (fields_autoplaced)
@@
     )
   )
+  (symbol (lib_id "Device:R") (at 67.31 172.72 90) (unit 1)
+    (in_bom yes) (on_board yes) (dnp no) (fields_autoplaced)
+    (property "Reference" "R8" (at 67.31 166.37 90)
+      (effects (font (size 1.27 1.27)))
+    )
+    (property "Value" "R" (at 67.31 168.91 90)
+      (effects (font (size 1.27 1.27)))
+    )
+    (property "Footprint" "Resistor_SMD:R_0805_2012Metric" (at 67.31 174.498 90)
+      (effects (font (size 1.27 1.27)) hide)
+    )
+    (property "Datasheet" "~" (at 67.31 172.72 0)
+      (effects (font (size 1.27 1.27)) hide)
+    )
+    (pin "1")
+    (pin "2")
+    (instances
+      (project "esp_espboy"
+        (path "/23d6f766-c6b7-4667-9a65-4887bf263ea9"
+          (reference "R8") (unit 1)
+        )
+      )
+    )
+  )
   (symbol (lib_id "esp_example_symbols:D2FS-FL-N-A") (at 167.64 120.65 0) (unit 1)
     (in_bom yes) (on_board yes) (dnp no) (fields_autoplaced)
@@
     )
   )
+  (symbol (lib_id "Device:C") (at 62.23 182.88 90) (unit 1)
+    (in_bom yes) (on_board yes) (dnp no) (fields_autoplaced)
+    (property "Reference" "C5" (at 62.23 175.26 90)
+      (effects (font (size 1.27 1.27)))
+    )
+    (property "Value" "C" (at 62.23 177.8 90)
+      (effects (font (size 1.27 1.27)))
+    )
+    (property "Footprint" "Capacitor_SMD:C_0805_2012Metric" (at 66.04 181.9148 0)
+      (effects (font (size 1.27 1.27)) hide)
+    )
+    (property "Datasheet" "~" (at 62.23 182.88 0)
+      (effects (font (size 1.27 1.27)) hide)
+    )
+    (pin "2")
+    (pin "1")
+    (instances
+      (project "esp_espboy"
+        (path "/23d6f766-c6b7-4667-9a65-4887bf263ea9"
+          (reference "C5") (unit 1)
+        )
+      )
+    )
+  )
   (symbol (lib_id "power:GND") (at 120.65 120.65 180) (unit 1)
     (in_bom yes) (on_board yes) (dnp no) (fields_autoplaced)
@@
         (path "/23d6f766-c6b7-4667-9a65-4887bf263ea9"
           (reference "R1") (unit 1)
+        )
+      )
+    )
+  )
+  (symbol (lib_id "Device:R") (at 19.05 124.46 0) (unit 1)
+    (in_bom yes) (on_board yes) (dnp no) (fields_autoplaced)
+    (property "Reference" "R5" (at 21.59 123.19 0)
+      (effects (font (size 1.27 1.27)) (justify left))
+    )
+    (property "Value" "R" (at 21.59 125.73 0)
+      (effects (font (size 1.27 1.27)) (justify left))
+    )
+    (property "Footprint" "Resistor_SMD:R_0805_2012Metric" (at 17.272 124.46 90)
+      (effects (font (size 1.27 1.27)) hide)
+    )
+    (property "Datasheet" "~" (at 19.05 124.46 0)
+      (effects (font (size 1.27 1.27)) hide)
+    )
+    (pin "1")
+    (pin "2")
+    (instances
+      (project "esp_espboy"
+        (path "/23d6f766-c6b7-4667-9a65-4887bf263ea9"
+          (reference "R5") (unit 1)
         )
       )
@@
     )
   )
+  (symbol (lib_id "Device:R") (at 67.31 167.64 90) (unit 1)
+    (in_bom yes) (on_board yes) (dnp no) (fields_autoplaced)
+    (property "Reference" "R6" (at 67.31 161.29 90)
+      (effects (font (size 1.27 1.27)))
+    )
+    (property "Value" "R" (at 67.31 163.83 90)
+      (effects (font (size 1.27 1.27)))
+    )
+    (property "Footprint" "Resistor_SMD:R_0805_2012Metric" (at 67.31 169.418 90)
+      (effects (font (size 1.27 1.27)) hide)
+    )
+    (property "Datasheet" "~" (at 67.31 167.64 0)
+      (effects (font (size 1.27 1.27)) hide)
+    )
+    (pin "1")
+    (pin "2")
+    (instances
+      (project "esp_espboy"
+        (path "/23d6f766-c6b7-4667-9a65-4887bf263ea9"
+          (reference "R6") (unit 1)
+        )
+      )
+    )
+  )
   (symbol (lib_id "Device:R") (at 55.88 54.61 0) (unit 1)
     (in_bom yes) (on_board yes) (dnp no) (fields_autoplaced)
@@
         )
       )
+    )
+  )
+  (symbol (lib_id "Device:R") (at 22.86 124.46 0) (unit 1)
+    (in_bom yes) (on_board yes) (dnp no) (fields_autoplaced)
+    (property "Reference" "R3" (at 25.4 123.19 0)
+      (effects (font (size 1.27 1.27)) (justify left))
+    )
+    (property "Value" "R" (at 25.4 125.73 0)
+      (effects (font (size 1.27 1.27)) (justify left))
+    )
+    (property "Footprint" "Resistor_SMD:R_0805_2012Metric" (at 21.082 124.46 90)
+      (effects (font (size 1.27 1.27)) hide)
+    )
+    (property "Datasheet" "~" (at 22.86 124.46 0)
+      (effects (font (size 1.27 1.27)) hide)
+    )
+    (pin "1")
+    (pin "2")
+    (instances
+      (project "esp_espboy"
+        (path "/23d6f766-c6b7-4667-9a65-4887bf263ea9"
+          (reference "R3") (unit 1)
+        )
+      )
+    )
+  )
+  (symbol (lib_id "Device:R") (at 67.31 170.18 90) (unit 1)
+    (in_bom yes) (on_board yes) (dnp no) (fields_autoplaced)
+    (property "Reference" "R7" (at 67.31 163.83 90)
+      (effects (font (size 1.27 1.27)))
+    )
+    (property "Value" "R" (at 67.31 166.37 90)
+      (effects (font (size 1.27 1.27)))
+    )
+    (property "Footprint" "Resistor_SMD:R_0805_2012Metric" (at 67.31 171.958 90)
+      (effects (font (size 1.27 1.27)) hide)
+    )
+    (property "Datasheet" "~" (at 67.31 170.18 0)
+      (effects (font (size 1.27 1.27)) hide)
+    )
+    (pin "1")
+    (pin "2")
+    (instances
+      (project "esp_espboy"
+        (path "/23d6f766-c6b7-4667-9a65-4887bf263ea9"
+          (reference "R7") (unit 1)
+        )
+      )
