File: KiCAD_designs/esp_examples/App_audio/compare_result/comparison.kicad_pcb (KiCad board)
At the start: 2 copper layers, 57 x 72 mm, 26 parts, among them J1 B4B-ZR-SM4-TFT_LF__SN_, J2 B2B-PH-SM4-TBLFSN, J3 Conn_01x02_Pin, J4 B4B-ZR-SM4-TFT_LF__SN_, J5 Conn_01x02_Pin, J6 B7B-ZR-SM4-TFT_LF__SN_, SW2 RS-282G05A3-SM RT, SW3 RS-282G05A3-SM RT, U1 ESP-12F, U2 AMS1117-3.3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

Commit message: cam_roller_arduino
Parts:
- removed J4: B4B-ZR-SM4-TFT_LF__SN_, esp_lib:JST_B4B-ZR-SM4-TFT_LF__SN_
- removed J6: B7B-ZR-SM4-TFT_LF__SN_, esp_lib:B7B-ZR-SM4-TBLFSN_JST
- removed S1: up, esp_lib:switch
- removed S2: down, esp_lib:switch
- removed S3: left, esp_lib:switch
- removed S4: right, esp_lib:switch
- removed S5: A, esp_lib:switch
- removed S6: B, esp_lib:switch
- removed S7: RL, esp_lib:switch
- removed S8: RR, esp_lib:switch
- added C10: 1u, Capacitor_SMD:C_0805_2012Metric, F.Cu at (47.7, 51.1)
- added C5: 0.47u, Capacitor_SMD:C_0805_2012Metric, F.Cu at (73.2, 35.0)
- added C6: 0.1u, Capacitor_SMD:C_0805_2012Metric, F.Cu at (59.8, 51.2)
- added C7: 1u, Capacitor_SMD:C_0805_2012Metric, F.Cu at (41.7, 51.1)
- added C8: 470u, esp_lib:CAP_EEEFP1C471AL, F.Cu at (88.9, 50.1)
- added C9: 1u, Capacitor_SMD:C_0805_2012Metric, F.Cu at (44.7, 51.1)
- added P1: S3B-ZR-SM4A-TF, esp_lib:JST_S3B-ZR-SM4A-TF, F.Cu at (54.8, 48.7)
- added SW1: RS-282G05A3-SM RT, esp_lib:RS-282G05A3-SM RT_CNK, F.Cu at (46.8, 45.0)
- J1: value B4B-ZR-SM4-TFT_LF__SN_ -> B2B-PH-SM4-TBLFSN; footprint esp_lib:JST_B4B-ZR-SM4-TFT_LF__SN_ -> esp_lib:B2B-PH-SM4-TBLFSN_JST
- U3: value MCP23017-E_SO -> PAM8403DR; footprint esp_lib:MCP23017 -> esp_lib:PAM8403
- moved U3 25.7 mm to (66.8, 51.3), turned to -90 degrees
- moved J1 5.50 mm to (77.5, 50.5), turned to 0 degrees
Connections:
- net Net-(J3-Pin_1) renamed /INL
- J1 pad 1: VCC -> Net-(U3-+OUT_L)
- J1 pad 2: GND -> Net-(U3--OUT_L)
- J1 pad 3: /SCK_mcp -> (no net)
- J1 pad 4: /SDA_mcp -> (no net)
- U1 pad 19: /SDA_mcp -> unconnected-(U1-GPIO4-Pad19)
- U1 pad 20: /SCK_mcp -> unconnected-(U1-GPIO5-Pad20)
- U1 pad 4: /AO -> unconnected-(U1-GPIO16-Pad4)
- U1 pad 5: /SDA_screen -> unconnected-(U1-GPIO14-Pad5)
- U1 pad 6: /CS -> Net-(U1-GPIO12)
- U1 pad 7: /SCK_screen -> unconnected-(U1-GPIO13-Pad7)
- U3 pad 1: unconnected-(U3-GPB0-Pad1) -> Net-(U3-+OUT_L)
- U3 pad 10: GND -> unconnected-(U3-INR-Pad10)
- U3 pad 11: (no net) -> GND
- U3 pad 12: /SCK_mcp -> VCC
- U3 pad 13: /SDA_mcp -> VCC
- U3 pad 14: (no net) -> unconnected-(U3--OUT_R-Pad14)
- U3 pad 15: unconnected-(U3-A0-Pad15) -> GND
- U3 pad 2: unconnected-(U3-GPB1-Pad2) -> GND
- U3 pad 3: unconnected-(U3-GPB2-Pad3) -> Net-(U3--OUT_L)
- U3 pad 4: unconnected-(U3-GPB3-Pad4) -> VCC
- U3 pad 5: unconnected-(U3-GPB4-Pad5) -> VCC
- U3 pad 6: unconnected-(U3-GPB5-Pad6) -> VCC
- U3 pad 7: unconnected-(U3-GPB6-Pad7) -> Net-(U3-INL)
- U3 pad 8: unconnected-(U3-GPB7-Pad8) -> Net-(U3-VREF)
- U3 pad 9: VCC -> (no net)
Routing:
- net /B: track 53.9 -> 0.00 mm
- net /SCK_mcp: track 49.6 -> 0.00 mm
- net VCC: track 213.8 -> 164.2 mm
- net /SDA_mcp: track 47.8 -> 0.00 mm
- net /RR: track 43.6 -> 0.00 mm
- net /A: track 40.3 -> 0.00 mm
- net Net-(C5-Pad2): track 0.00 -> 29.2 mm
- net /RL: track 29.1 -> 0.00 mm
- net /left: track 26.6 -> 0.00 mm
- net /AO: track 26.5 -> 0.00 mm
- net /SDA_screen: track 25.3 -> 0.00 mm
- net /CS: track 23.3 -> 0.00 mm
- net /SCK_screen: track 21.8 -> 0.00 mm
- net /down: track 20.4 -> 0.00 mm
- net /up: track 19.6 -> 0.00 mm
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Other:
- board size 57 x 72 mm -> 57 x 33 mm
