File: KiCAD_designs/esp_examples/App_cam_roller/compare_result/comparison.kicad_pcb (KiCad board)
At the start: 2 copper layers, 57 x 37 mm, 21 parts, among them J1 B2B-PH-SM4-TBLFSN, J2 B2B-PH-SM4-TBLFSN, J3 Conn_01x02_Pin, J4 B2B-PH-SM4-TBLFSN, J5 Conn_01x02_Pin, SW2 RS-282G05A3-SM RT, SW3 RS-282G05A3-SM RT, U1 ESP-12F, U2 AMS1117-3.3, U3 MX1508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

Commit message: cam_roller_arduino
Parts:
- added R4: R, Resistor_SMD:R_0805_2012Metric, F.Cu at (46.2, 40.3)
- moved R1 0.49 mm to (46.2, 36.2)
Connections:
- U1 pad 3: unconnected-(U1-EN-Pad3) -> Net-(U1-EN)
Routing:
- net Net-(U1-EN): track 0.00 -> 14.9 mm
- net /RST: track 20.2 -> 18.8 mm
- net VCC: track 190.7 -> 191.4 mm
