File: KiCAD_designs/workflow_example/workflow_1/workflow_1.kicad_sch (KiCad schematic)
At the start: 5 parts, among them J1 B2B-PH-SM4-TBLFSN, SW1 CUS-12TB, U1 ATTINY45-20SU

Commit message: workflow example
Connections:
- net LED: now also U1.6 (PB1); no longer U1.5 (PB0)
Changed lines of the file:
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@@
     (effects (font (size 1.27 1.27)) (justify left bottom))
   )
-  (label "LED" (at 74.93 74.93 180) (fields_autoplaced)
+  (label "GND" (at 125.095 93.345 180) (fields_autoplaced)
     (effects (font (size 1.27 1.27)) (justify right bottom))
   )
-  (label "GND" (at 125.095 93.345 180) (fields_autoplaced)
+  (label "LED" (at 74.93 77.47 180) (fields_autoplaced)
     (effects (font (size 1.27 1.27)) (justify right bottom))
   )
@@
     (pin "2")
     (instances
-      (project "workflow"
+      (project "workflow_1"
         (path "/f73d03d9-3aa3-47b4-8285-cbe7ff2a4073"
           (reference "D1") (unit 1)
@@
     (pin "2")
     (instances
-      (project "workflow"
+      (project "workflow_1"
         (path "/f73d03d9-3aa3-47b4-8285-cbe7ff2a4073"
           (reference "R1") (unit 1)
@@
     (pin "2")
     (instances
-      (project "workflow"
+      (project "workflow_1"
         (path "/f73d03d9-3aa3-47b4-8285-cbe7ff2a4073"
           (reference "J1") (unit 1)
@@
     (pin "1")
     (instances
-      (project "workflow"
+      (project "workflow_1"
         (path "/f73d03d9-3aa3-47b4-8285-cbe7ff2a4073"
           (reference "SW1") (unit 1)
@@
     (pin "3")
     (instances
-      (project "workflow"
+      (project "workflow_1"
         (path "/f73d03d9-3aa3-47b4-8285-cbe7ff2a4073"
           (reference "U1") (unit 1)
