File: KiCAD_designs/workflow_example/workflow_1/compare_result/comparison.kicad_pcb (KiCad board)
At the start: 2 copper layers, 21 x 18 mm, 5 parts, among them J1 B2B-PH-SM4-TBLFSN, SW1 CUS-12TB, U1 ATTINY45-20SU

Commit message: workflow example
Connections:
- U1 pad 5: /LED -> unconnected-(U1-PB0-Pad5)
- U1 pad 6: unconnected-(U1-PB1-Pad6) -> /LED
Routing:
- net /LED: track 5.41 -> 6.46 mm
