File: KiCAD_designs/cat_ball/cat_ball.kicad_sch (KiCad schematic)
At the start: 35 parts, among them J1 B2B-PH-SM4-TBLFSN, J2 B2B-PH-SM4-TBLFSN, U1 ATMEGA328P-AU, U2 MX1508

Commit message: catball thicker traces
Parts:
- J1, J2: footprint esp_lib:B2B-PH-SM4-TBLFSN_JST -> IO_watch_cat_ball:B2B-PH-SM4-TBLFSN_JST
- U2: footprint esp_lib:MX1508 -> IO_watch_cat_ball:MX1508
Changed lines of the file:
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@@
       (effects (font (size 1.27 1.27)))
     )
-    (property "Footprint" "esp_lib:MX1508" (at 200.66 104.14 0)
+    (property "Footprint" "IO_watch_cat_ball:MX1508" (at 200.66 104.14 0)
       (effects (font (size 1.27 1.27)) (justify bottom) hide)
     )
@@
       (effects (font (size 1.524 1.524)))
     )
-    (property "Footprint" "esp_lib:B2B-PH-SM4-TBLFSN_JST" (at 217.17 81.28 0)
+    (property "Footprint" "IO_watch_cat_ball:B2B-PH-SM4-TBLFSN_JST" (at 217.17 81.28 0)
       (effects (font (size 1.27 1.27) italic) hide)
     )
@@
       (effects (font (size 1.524 1.524)))
     )
-    (property "Footprint" "esp_lib:B2B-PH-SM4-TBLFSN_JST" (at 173.99 123.19 0)
+    (property "Footprint" "IO_watch_cat_ball:B2B-PH-SM4-TBLFSN_JST" (at 173.99 123.19 0)
       (effects (font (size 1.27 1.27) italic) hide)
     )
